File: efm32-board.kicad_pcb (KiCad board)
At the start: 2 copper layers, 18.8 x 51.8 mm, 32 parts, among them J1 Conn_01x20, J2 Conn_01x20, J3 USB_OTG, J4 SWD, J5 Conn_01x20, J6 Conn_01x20, SW1 reset, SW2 reset, U1 EFM32HG-48LQFP, U2 SPX3819M5-L-3-3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

Commit message: Add copyright and logo
Signed-off-by: Martin Ribelotta <martinribelotta@gmail.com>
Parts:
- added G102: LOGO_CIAA, footprints:LOGO-CIAA, B.Cu at (127.4, 76.1)
Other:
- board text added: "copyright © by Martin Ribelotta"
- board text added: "licenced under BSD-3 clauses & CIAA-HW"
Changed lines of the file:
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@@
   (general
     (thickness 1.6)
-    (drawings 8)
+    (drawings 20)
     (tracks 671)
     (zones 0)
-    (modules 32)
+    (modules 33)
     (nets 51)
   )
@@
     (add_net "Net-(R2-Pad1)")
   )
+  (module footprints:LOGO-CIAA (layer B.Cu)
+    (at 127.438 76.085 90)
+    (fp_text reference G102 (at 0 -4.99364 90) (layer B.SilkS) hide
+      (effects (font (size 0.7112 0.4572) (thickness 0.1143)) (justify mirror))
+    )
+    (fp_text value LOGO_CIAA (at 0 4.99364 90) (layer B.SilkS) hide
+      (effects (font (thickness 0.3048)) (justify mirror))
+    )
+    (fp_poly (pts (xy 4.23418 -4.23418) (xy 0 -4.23418) (xy -4.23164 -4.23418) (xy -4.23164 0)
+      (xy -4.23164 4.23164) (xy 0 4.23164) (xy 4.23418 4.23164) (xy 4.23418 0.43434)
+      (xy 4.23418 -3.3655) (xy 3.8735 -3.28676) (xy 3.47218 -3.2131) (xy 2.9464 -3.1369)
+      (xy 2.37236 -3.06578) (xy 2.37236 -2.3749) (xy 2.34188 -2.24536) (xy 2.26314 -2.00406)
+      (xy 2.14884 -1.69418) (xy 2.02184 -1.36144) (xy 1.8923 -1.04648) (xy 1.84912 -0.9525)
+      (xy 1.72466 -0.73152) (xy 1.59766 -0.60706) (xy 1.55448 -0.59436) (xy 1.46304 -0.64008)
+      (xy 1.48082 -0.74168) (xy 1.53162 -0.8763) (xy 1.6256 -1.12522) (xy 1.7399 -1.43764)
+      (xy 1.86182 -1.7653) (xy 1.97104 -2.06756) (xy 2.05232 -2.29108) (xy 2.07518 -2.3495)
+      (xy 2.16154 -2.43332) (xy 2.28854 -2.4511) (xy 2.36728 -2.39522) (xy 2.37236 -2.3749)
+      (xy 2.37236 -3.06578) (xy 2.34442 -3.06324) (xy 1.92786 -3.01752) (xy 1.92786 -2.42062)
+      (xy 1.92278 -2.33934) (xy 1.87706 -2.18186) (xy 1.78308 -1.92532) (xy 1.6383 -1.54178)
+      (xy 1.58242 -1.397) (xy 1.43002 -1.01854) (xy 1.30048 -0.76454) (xy 1.18618 -0.63754)
+      (xy 1.07188 -0.64262) (xy 0.94742 -0.78994) (xy 0.8001 -1.0795) (xy 0.61722 -1.52146)
+      (xy 0.46228 -1.92786) (xy 0.35814 -2.20726) (xy 0.31496 -2.36728) (xy 0.3302 -2.4384)
+      (xy 0.39624 -2.45618) (xy 0.41656 -2.45618) (xy 0.51054 -2.413) (xy 0.61468 -2.26568)
+      (xy 0.73914 -1.99644) (xy 0.84836 -1.71958) (xy 1.12776 -0.98044) (xy 1.29286 -1.44272)
+      (xy 1.45796 -1.88214) (xy 1.5875 -2.18186) (xy 1.69164 -2.3622) (xy 1.78308 -2.44348)
+      (xy 1.83388 -2.45618) (xy 1.89484 -2.4511) (xy 1.92786 -2.42062) (xy 1.92786 -3.01752)
+      (xy 1.70942 -2.9972) (xy 1.08966 -2.94132) (xy 0.53086 -2.90322) (xy 0.07874 -2.88544)
+      (xy 0 -2.88544) (xy 0 -1.69926) (xy 0 -1.524) (xy -0.00254 -1.1176)
+      (xy -0.01016 -0.84836) (xy -0.03302 -0.69342) (xy -0.07366 -0.61722) (xy -0.13716 -0.59436)
+      (xy -0.16764 -0.59436) (xy -0.24384 -0.60452) (xy -0.2921 -0.65532) (xy -0.32004 -0.77724)
+      (xy -0.33274 -0.99822) (xy -0.33782 -1.34874) (xy -0.33782 -1.524) (xy -0.33528 -1.93294)
+      (xy -0.32766 -2.19964) (xy -0.3048 -2.35712) (xy -0.26416 -2.43078) (xy -0.20066 -2.45364)
+      (xy -0.16764 -2.45618) (xy -0.09398 -2.44602) (xy -0.04572 -2.39268) (xy -0.01778 -2.27076)
+      (xy -0.00508 -2.04978) (xy 0 -1.69926) (xy 0 -2.88544) (xy -0.4191 -2.8956)
+      (xy -0.94488 -2.92862) (xy -1.016 -2.9337) (xy -1.016 -0.75438) (xy -1.08966 -0.62992)
+      (xy -1.2827 -0.56642) (xy -1.55448 -0.56896) (xy -1.74244 -0.60452) (xy -2.07264 -0.77216)
+      (xy -2.28092 -1.05918) (xy -2.36728 -1.45542) (xy -2.36982 -1.54178) (xy -2.35204 -1.8288)
+      (xy -2.2733 -2.02692) (xy -2.11836 -2.21234) (xy -1.93548 -2.36982) (xy -1.75514 -2.4384)
+      (xy -1.50114 -2.44094) (xy -1.46304 -2.4384) (xy -1.18618 -2.4003) (xy -1.0541 -2.3241)
+      (xy -1.03378 -2.27838) (xy -1.05156 -2.18948) (xy -1.18364 -2.17424) (xy -1.26492 -2.18186)
+      (xy -1.63576 -2.17424) (xy -1.91008 -2.03962) (xy -2.06756 -1.79832) (xy -2.09296 -1.46558)
+      (xy -2.07772 -1.36906) (xy -1.94564 -1.06426) (xy -1.71704 -0.89408) (xy -1.3843 -0.85852)
+      (xy -1.3589 -0.86106) (xy -1.13284 -0.86868) (xy -1.03378 -0.8255) (xy -1.016 -0.75438)
+      (xy -1.016 -2.9337) (xy -1.51892 -2.97688) (xy -2.07518 -3.0353) (xy -2.19964 -3.05054)
+      (xy -2.82194 -3.12928) (xy -3.29438 -3.19278) (xy -3.63982 -3.24104) (xy -3.87604 -3.28422)
+      (xy -4.0259 -3.31978) (xy -4.10718 -3.35788) (xy -4.1402 -3.39852) (xy -4.14782 -3.44678)
+      (xy -4.14782 -3.44932) (xy -4.10718 -3.5306) (xy -3.95478 -3.53822) (xy -3.8735 -3.52806)
+      (xy -3.1369 -3.42392) (xy -2.2733 -3.35026) (xy -1.31064 -3.30454) (xy -0.2921 -3.28676)
+      (xy 0.75184 -3.29692) (xy 1.78054 -3.33502) (xy 2.76352 -3.40106) (xy 3.6576 -3.49504)
+      (xy 3.8735 -3.52552) (xy 4.09956 -3.56616) (xy 4.2037 -3.63474) (xy 4.23164 -3.78206)
+      (xy 4.23418 -3.90398) (xy 4.23418 -4.23418) (xy 4.23418 -4.23418)) (layer B.SilkS) (width 0.00254))
+  )
   (module Pin_Headers:Pin_Header_Straight_2x02_Pitch2.54mm_SMD (layer F.Cu)
     (at 123.358 81.465 270)
@@
     (tags "Surface mounted pin header SMD 2x02 2.54mm double row")
     (attr smd)
-    (fp_text reference J4 (at 0 -3.6 270) (layer F.SilkS)
+    (fp_text reference J4 (at 4.85 0 270) (layer F.SilkS)
       (effects (font (size 1 1) (thickness 0.15)))
     )
@@
     (tags "capacitor 0603")
     (attr smd)
-    (fp_text reference C9 (at -2.48 0.2) (layer F.SilkS)
+    (fp_text reference C9 (at 0.61 -1.32) (layer F.SilkS)
       (effects (font (size 1 1) (thickness 0.15)))
     )
@@
     (tags "capacitor 0603")
     (attr smd)
-    (fp_text reference C2 (at 2.37 0 270) (layer F.SilkS)
+    (fp_text reference C2 (at 0.72 -1.36 270) (layer F.SilkS)
       (effects (font (size 1 1) (thickness 0.15)))
     )
@@
     (tags "capacitor 0603")
     (attr smd)
-    (fp_text reference C6 (at 0.4 -1.31 90) (layer F.SilkS)
+    (fp_text reference C6 (at 0.12 -1.25 90) (layer F.SilkS)
       (effects (font (size 1 1) (thickness 0.15)))
     )
@@
     (tags "capacitor 0603")
     (attr smd)
-    (fp_text reference C12 (at 0.06 1.43 90) (layer F.SilkS)
+    (fp_text reference C12 (at 0.05 1.51 90) (layer F.SilkS)
       (effects (font (size 1 1) (thickness 0.15)))
     )
@@
     )
   )
+  (gr_arc (start 123.868 112.675) (end 125.908 107.905) (angle -45.68445884) (layer F.SilkS) (width 0.15))
+  (gr_line (start 125.408 105.175) (end 125.948 106.965) (layer F.SilkS) (width 0.3))
+  (gr_line (start 124.748 105.185) (end 125.288 106.975) (layer F.SilkS) (width 0.3))
+  (gr_line (start 124.748 105.185) (end 124.208 106.965) (layer F.SilkS) (width 0.3))
+  (gr_line (start 123.728 105.185) (end 123.728 106.965) (layer F.SilkS) (width 0.3))
+  (gr_arc (start 122.560995 106.072005) (end 123.188 105.445) (angle -270) (layer F.SilkS) (width 0.3))
+  (gr_line (start 121.31 108.63) (end 121.31 103.63) (layer F.SilkS) (width 0.15))
+  (gr_line (start 126.31 108.63) (end 121.31 108.63) (layer F.SilkS) (width 0.15))
+  (gr_line (start 126.31 103.63) (end 126.31 108.63) (layer F.SilkS) (width 0.15))
+  (gr_line (start 121.31 103.63) (end 126.31 103.63) (layer F.SilkS) (width 0.15))
+  (gr_text "licenced under\nBSD-3 clauses\n& CIAA-HW" (at 123.638 115.155 270) (layer B.SilkS)
+    (effects (font (size 1 1) (thickness 0.2)) (justify mirror))
+  )
+  (gr_text "copyright © by\nMartin Ribelotta" (at 131.318 114.985 270) (layer B.SilkS)
+    (effects (font (size 1 1) (thickness 0.2)) (justify mirror))
+  )
   (gr_text PWR (at 126.818 120.755 90) (layer F.SilkS)
